File: PTP_project1/PTP_project1.kicad_pcb (KiCad board)
At the start: 2 copper layers, 45 parts, among them J1 Screw_Terminal_01x02, SW1 SW_MEC_5G, SW2 SW_SPDT_312, U1 LM2574N-5, U2 4027, U3 4027, U4 74LS47, U5 HDSP-7401, U6 SN74LVC1G11, U7 NE555P

Commit message: lv8
Parts:
- moved R19 86.2 mm to (106.0, 81.5), turned to 90 degrees
- moved R20 86.1 mm to (106.0, 75.0), turned to 90 degrees
- moved U7 82.7 mm to (110.2, 74.7)
- moved U5 81.4 mm to (192.5, 67.0)
- moved R6 79.7 mm to (185.5, 81.0), turned to 0 degrees
- moved R8 79.6 mm to (185.5, 84.5), turned to 0 degrees
- moved R9 53.6 mm to (159.5, 91.0)
- moved U6 45.5 mm to (132.5, 68.0)
- moved C5 39.9 mm to (122.5, 80.0)
- moved R7 39.0 mm to (155.0, 91.0), turned to 90 degrees
- moved R13 37.6 mm to (151.0, 91.0), turned to 90 degrees
- moved C4 35.2 mm to (114.0, 89.5), turned to 0 degrees
- moved R10 35.0 mm to (164.0, 91.0), turned to 90 degrees
- moved R5 33.7 mm to (185.5, 77.5)
- moved R11 29.4 mm to (168.0, 91.0), turned to 90 degrees
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Routing:
- net +5V: track 0.00 -> 265.7 mm, vias 0 -> 16
- net GND: track 0.00 -> 178.9 mm, vias 0 -> 2
- net Q3: track 0.00 -> 86.4 mm, vias 0 -> 4
- net Q0: track 0.00 -> 72.0 mm, vias 0 -> 2
- net Q1: track 0.00 -> 63.1 mm, vias 0 -> 2
- net Net-(U7-THR): track 0.00 -> 57.8 mm, vias 0 -> 4
- net Clock: track 0.00 -> 55.9 mm, vias 0 -> 2
- net VD: track 0.00 -> 55.2 mm, vias 0 -> 2
- net Net-(SW2-A): track 0.00 -> 39.8 mm, vias 0 -> 2
- net Net-(U4-BI): track 0.00 -> 38.2 mm, vias 0 -> 2
- net Q2: track 0.00 -> 36.9 mm, vias 0 -> 6
- net Net-(D4-K): track 0.00 -> 34.2 mm
- net Net-(U2A-J): track 0.00 -> 33.2 mm
- net Reset: track 0.00 -> 33.1 mm, vias 0 -> 4
- net 555: track 0.00 -> 28.6 mm, vias 0 -> 2
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- added copper zone on B.Cu, net GND

Commit message: lv9
Parts:
- moved R5 0.50 mm to (185.5, 77.0)
Routing:
- net GND: track 178.9 -> 194.0 mm
- net +5V: track 265.7 -> 274.2 mm
- net Net-(U3A-J): track 26.2 -> 28.8 mm
- net Net-(U3B-J): track 22.7 -> 25.3 mm
- net Net-(U2B-J): track 25.1 -> 27.7 mm
- net unconnected-(U5-DP-Pad7): track 1.15 -> 0.00 mm
Other:
- board outline added: 100 x 80 mm
- board text added: "PTP - BCD counter Gabriel Šolčić"
Changed lines of the file:
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@@
 			(usegerberattributes yes)
 			(usegerberadvancedattributes yes)
-			(creategerberjobfile yes)
+			(creategerberjobfile no)
 			(dashed_line_dash_ratio 12.000000)
 			(dashed_line_gap_ratio 3.000000)
@@
 			(outputformat 1)
 			(mirror no)
-			(drillshape 1)
+			(drillshape 0)
 			(scaleselection 1)
-			(outputdirectory "")
+			(outputdirectory "C:/Users/gsolcic/Documents/GitHub/PTP_Gabriel_Solcic_Project1/PTP_project1/Manufacturing/")
 		)
 	)
@@
 		(tags "resistor handsolder")
 		(property "Reference" "R14"
-			(at 0 -1.83 0)
+			(at -4.5 0 0)
 			(layer "F.SilkS")
 			(effects
@@
 		(tags "resistor handsolder")
 		(property "Reference" "R6"
-			(at 0 -1.5 0)
+			(at -4 -0.5 0)
 			(layer "F.SilkS")
 			(effects
@@
 		(tags "resistor handsolder")
 		(property "Reference" "R18"
-			(at 0 -1.83 0)
+			(at -4 -2 0)
 			(layer "F.SilkS")
 			(effects
@@
 	(footprint "Resistor_SMD:R_1206_3216Metric_Pad1.30x1.75mm_HandSolder"
 		(layer "F.Cu")
-		(at 185.5 77.5)
+		(at 185.5 77)
 		(descr "Resistor SMD 1206 (3216 Metric), square (rectangular) end terminal, IPC-7351 nominal with elongated pad for handsoldering. (Body size source: IPC-SM-782 page 72, https://www.pcb-3d.com/wordpress/wp-content/uploads/ipc-sm-782a_amendment_1_and_2.pdf), generated with kicad-footprint-generator")
 		(tags "resistor handsolder")
 		(property "Reference" "R5"
-			(at 0 -1.83 0)
+			(at -4 -0.5 0)
 			(layer "F.SilkS")
 			(effects
@@
 		(tags "resistor handsolder")
 		(property "Reference" "R17"
-			(at 0 -1.83 0)
+			(at -4 -2 0)
 			(layer "F.SilkS")
 			(effects
@@
 		(tags "resistor handsolder")
 		(property "Reference" "R16"
-			(at 0 -1.83 0)
+			(at -4.55 -2.5 0)
 			(layer "F.SilkS")
 			(effects
@@
 		(tags "resistor handsolder")
 		(property "Reference" "R8"
-			(at 0 -1.83 0)
+			(at -4 -0.5 0)
 			(layer "F.SilkS")
 			(effects
@@
 		(tags "resistor handsolder")
 		(property "Reference" "R15"
-			(at 0 -1.83 0)
+			(at -4.5 -1.5 0)
 			(layer "F.SilkS")
 			(effects
@@
 		(tags "switch SPDT")
 		(property "Reference" "SW2"
-			(at 3.99 -2.99 90)
+			(at -4.5 0 180)
 			(layer "F.SilkS")
 			(effects
@@
 		(stroke
 			(width 0.2)
-			(type default)
+			(type solid)
 		)
-		(layer "F.Cu")
+		(layer "Edge.Cuts")
 	)
 	(gr_line
@@
 		(stroke
 			(width 0.2)
-			(type default)
+			(type solid)
 		)
-		(layer "F.Cu")
+		(layer "Edge.Cuts")
 	)
 	(gr_arc
@@
 		(stroke
 			(width 0.2)
-			(type default)
+			(type solid)
 		)
-		(layer "F.Cu")
+		(layer "Edge.Cuts")
 	)
 	(gr_arc
@@
 		(stroke
 			(width 0.2)
-			(type default)
+			(type solid)
 		)
-		(layer "F.Cu")
+		(layer "Edge.Cuts")
 	)
 	(gr_line
@@
 		(stroke
 			(width 0.2)
-			(type default)
+			(type solid)
 		)
-		(layer "F.Cu")
+		(layer "Edge.Cuts")
 	)
 	(gr_arc
@@
 		(stroke
 			(width 0.2)
-			(type default)
+			(type solid)
 		)
-		(layer "F.Cu")
+		(layer "Edge.Cuts")
 	)
 	(gr_line
@@
 		(stroke
 			(width 0.2)
-			(type default)
+			(type solid)
 		)
-		(layer "F.Cu")
+		(layer "Edge.Cuts")
 	)
 	(gr_line
@@
 		(stroke
 			(width 0.2)
-			(type default)
+			(type solid)
+		)
+		(layer "Edge.Cuts")
+	)
+	(gr_text "PTP - BCD counter\nGabriel Šolčić"
+		(at 117.5 103 0)
+		(layer "F.SilkS")
+		(effects
+			(font
+				(size 2 1.5)
+				(thickness 0.2)
+			)
+			(justify left bottom)
 		)
-		(layer "F.Cu")
 	)
 	(segment
@@
 	)
 	(segment
+		(start 155.19 77.910768)
+		(end 155.19 78.35)
+		(width 0.2)
+		(layer "F.Cu")
+		(net 2)
+	)
+	(segment
 		(start 110.195 72.805)
 		(end 110.5 72.5)
@@
 	)
 	(segment
+		(start 148.309 79.389)
+		(end 148.309 75.353951)
+		(width 0.2)
+		(layer "F.Cu")
+		(net 2)
+	)
+	(segment
 		(start 151.75 100.75)
 		(end 148.5 97.5)
@@
 	)
 	(segment
+		(start 148.309 75.353951)
+		(end 148.953951 74.709)
+		(width 0.2)
+		(layer "F.Cu")
+		(net 2)
+	)
+	(segment
 		(start 138 91.5)
 		(end 136 89.5)
@@
 	)
 	(segment
+		(start 149.81 80.89)
+		(end 148.309 79.389)
+		(width 0.2)
+		(layer "F.Cu")
+		(net 2)
+	)
+	(segment
 		(start 118.749 41.847292)
 		(end 118.749 39.11963)
@@
 	)
 	(segment
+		(start 151.988232 74.709)
+		(end 155.19 77.910768)
+		(width 0.2)
+		(layer "F.Cu")
+		(net 2)
+	)
+	(segment
 		(start 123.9375 78.4375)
 		(end 122.5 78.4375)
@@
 		(net 2)
 	)
+	(segment
+		(start 148.953951 74.709)
+		(end 151.988232 74.709)
+		(width 0.2)
+		(layer "F.Cu")
+		(net 2)
+	)
 	(via
 		(at 130 70)
@@
 	)
 	(segment
+		(start 164 92.55)
+		(end 168 92.55)
+		(width 0.5)
+		(layer "F.Cu")
+		(net 3)
+	)
+	(segment
 		(start 192.5325 63.0325)
 		(end 188.5 59)
@@
 	)
 	(segment
+		(start 159.5 92.55)
+		(end 164 92.55)
+		(width 0.5)
+		(layer "F.Cu")
+		(net 3)
+	)
+	(segment
 		(start 120 75)
 		(end 121 76)
@@
 	)
 	(segment
+		(start 149.81 78.35)
+		(end 149.81 75.81)
+		(width 0.2)
+		(layer "F.Cu")
+		(net 23)
+	)
+	(segment
 		(start 152.5 85)
 		(end 152.5 76)
@@
 	)
 	(segment
+		(start 155.19 75.81)
+		(end 155.19 73.27)
+		(width 0.2)
+		(layer "F.Cu")
+		(net 24)
+	)
+	(segment
 		(start 160 85)
 		(end 160 73.5)
@@
 	)
 	(segment
+		(start 162.81 78.35)
+		(end 162.81 75.81)
+		(width 0.2)
+		(layer "F.Cu")
+		(net 25)
+	)
+	(segment
 		(start 192.5325 77.1425)
 		(end 192.5325 84.5175)
@@
 	)
 	(segment
-		(start 180 73)
-		(end 181 73)
-		(width 0.5)
-		(layer "B.Cu")
-		(net 30)
-	)
-	(segment
-		(start 181 73)
-		(end 181.5 73.5)
+		(start 179 83.5)
+		(end 179 74)
 		(width 0.5)
 		(layer "B.Cu")
@@
 	)
 	(segment
-		(start 179 83.5)
-		(end 179 74)
+		(start 179 74)
+		(end 179.5 73.5)
 		(width 0.5)
 		(layer "B.Cu")
@@
 	)
 	(segment
-		(start 179 74)
-		(end 180 73)
+		(start 179.5 73.5)
+		(end 181.5 73.5)
 		(width 0.5)
 		(layer "B.Cu")
@@
 	)
 	(segment
-		(start 181.14 68.19)
-		(end 183.45 70.5)
+		(start 175.81 68.19)
+		(end 177.62 70)
 		(width 0.5)
 		(layer "F.Cu")
@@
 	)
 	(segment
-		(start 175.81 68.19)
-		(end 181.14 68.19)
+		(start 177.62 70)
+		(end 182.95 70)
+		(width 0.5)
+		(layer "F.Cu")
+		(net 34)
+	)
+	(segment
+		(start 182.95 70)
+		(end 183.45 70.5)
 		(width 0.5)
 		(layer "F.Cu")
@@
 		(net 40)
 	)
-	(segment
-		(start 197.6125 74.6025)
-		(end 196.6025 74.6025)
-		(width 0.5)
-		(layer "F.Cu")
-		(net 45)
-	)
-	(segment
-		(start 196.6025 74.6025)
-		(end 196.5 74.5)
-		(width 0.5)
-		(layer "F.Cu")
-		(net 45)
-	)
 	(zone
